Commit message: construccion inicial inspiracion A1

File: urdf/spotmicro.urdf.xacro (robot description, xacro)
@@ -1,4 +1,5 @@
 <?xml version="1.0"?>
 <robot xmlns:xacro="http://www.ros.org/wiki/xacro" name="spotmicro_description">
+  <xacro:include filename="$(find spotmicro_description)/urdf/spotmicro.ros2_control.xacro"/>
   <material name="yellow">
     <color rgba="0.92 0.83 0.0 1"/>
@@ -29,4 +30,5 @@
   <xacro:property name="shiftx" value="0.093" />
   <xacro:property name="shifty" value="0.039" />
+  <xacro:property name="mesh_dir" value="file://$(find spotmicro_description)/meshes/visual" />
   <!-- Macros -->
   <xacro:macro name="gen_shoulder" params="name left">
@@ -35,5 +37,5 @@
         <xacro:if value="${left}">
         <geometry>
-          <mesh filename="package://chaski_rviz/urdf/stl/lshoulder.stl" scale="0.001 0.001 0.001"/>
+          <mesh filename="${mesh_dir}/lshoulder.stl" scale="0.001 0.001 0.001"/>
         </geometry>
         <origin rpy="0 0 3.14159" xyz="0.135 0.015 -0.01"/>
@@ -41,5 +43,5 @@
         <xacro:unless value="${left}">
         <geometry>
-          <mesh filename="package://chaski_rviz/urdf/stl/rshoulder.stl" scale="0.001 0.001 0.001"/>
+          <mesh filename="${mesh_dir}/rshoulder.stl" scale="0.001 0.001 0.001"/>
         </geometry>
         <origin rpy="0 0 3.14159" xyz="0.135 0.095 -0.01"/>
@@ -74,5 +76,5 @@
         <xacro:if value="${left}">
         <geometry>
-          <mesh filename="package://chaski_rviz/urdf/stl/larm_cover.stl" scale="0.001 0.001 0.001"/>
+          <mesh filename="${mesh_dir}/larm_cover.stl" scale="0.001 0.001 0.001"/>
         </geometry>
         <origin rpy="0 -0.139 3.14159" xyz="0.130 -0.040 -0.025"/>
@@ -80,5 +82,5 @@
         <xacro:unless value="${left}">
         <geometry>
-          <mesh filename="package://chaski_rviz/urdf/stl/rarm_cover.stl" scale="0.001 0.001 0.001"/>
+          <mesh filename="${mesh_dir}/rarm_cover.stl" scale="0.001 0.001 0.001"/>
         </geometry>
         <origin rpy="0 -0.139 3.14159" xyz="0.130 0.15 -0.025"/>
@@ -91,5 +93,5 @@
         <xacro:if value="${left}">
         <geometry>
-          <mesh filename="package://chaski_rviz/urdf/stl/larm.stl" scale="0.001 0.001 0.001"/>
+          <mesh filename="${mesh_dir}/larm.stl" scale="0.001 0.001 0.001"/>
         </geometry>
         <origin rpy="0 -0.139 3.14159" xyz="0.130 -0.040 -0.025"/>
@@ -97,5 +99,5 @@
         <xacro:unless value="${left}">
         <geometry>
-          <mesh filename="package://chaski_rviz/urdf/stl/rarm.stl" scale="0.001 0.001 0.001"/>
+          <mesh filename="${mesh_dir}/rarm.stl" scale="0.001 0.001 0.001"/>
         </geometry>
         <origin rpy="0 -0.139 3.14159" xyz="0.130 0.15 -0.025"/>
@@ -140,5 +142,5 @@
         <xacro:if value="${left}">
         <geometry>
-          <mesh filename="package://chaski_rviz/urdf/stl/lfoot.stl" scale="0.001 0.001 0.001"/>
+          <mesh filename="${mesh_dir}/lfoot.stl" scale="0.001 0.001 0.001"/>
         </geometry>
         <origin rpy="0 0 3.14159" xyz="0.120 -0.04 0.1"/>
@@ -146,5 +148,5 @@
         <xacro:unless value="${left}">
         <geometry>
-          <mesh filename="package://chaski_rviz/urdf/stl/rfoot.stl" scale="0.001 0.001 0.001"/>
+          <mesh filename="${mesh_dir}/rfoot.stl" scale="0.001 0.001 0.001"/>
         </geometry>
         <origin rpy="0 0 3.14159" xyz="0.120 0.15 0.1"/>
@@ -178,5 +180,5 @@
       <visual>
         <geometry>
-        <mesh filename="package://chaski_rviz/urdf/stl/foot.stl" scale="0.001 0.001 0.001"/>
+        <mesh filename="${mesh_dir}/foot.stl" scale="0.001 0.001 0.001"/>
         </geometry>
         <origin rpy="0 -0.40010 3.14159" xyz="0.00 0.01 0.015"/>
@@ -223,5 +225,5 @@
     <visual>
       <geometry>
-        <mesh filename="package://chaski_rviz/urdf/stl/mainbody.stl" scale="0.001 0.001 0.001"/>
+        <mesh filename="${mesh_dir}/mainbody.stl" scale="0.001 0.001 0.001"/>
       </geometry>
       <material name="black"/>
@@ -243,5 +245,5 @@
     <visual>
       <geometry>
-        <mesh filename="package://chaski_rviz/urdf/stl/rplidar_main.STL" scale="0.001 0.001 0.001"/>
+        <mesh filename="${mesh_dir}/rplidar_main.STL" scale="0.001 0.001 0.001"/>
       </geometry>
       <material name="black"/>
@@ -267,5 +269,5 @@
     <visual>
       <geometry>
-        <mesh filename="package://chaski_rviz/urdf/stl/backpart.stl" scale="0.001 0.001 0.001"/>
+        <mesh filename="${mesh_dir}/backpart.stl" scale="0.001 0.001 0.001"/>
       </geometry>
       <origin rpy="0 0 3.14159" xyz="0.04 0.055 -0.010"/>
@@ -290,5 +292,5 @@
     <visual>
       <geometry>
-        <mesh filename="package://chaski_rviz/urdf/stl/frontpart.stl" scale="0.001 0.001 0.001"/>
+        <mesh filename="${mesh_dir}/frontpart.stl" scale="0.001 0.001 0.001"/>
       </geometry>
       <origin rpy="0 0 3.14159" xyz="0.040 0.055 -0.010"/>

Commit message: Integracion de sensor IMU

File: urdf/spotmicro.urdf.xacro (robot description, xacro)
@@ -19,4 +19,5 @@
   <xacro:property name="lidar_width" value="0.0577" />
   <xacro:property name="lidar_height" value="0.070" />
+  <xacro:property name="imu_size" value="0.001" />
   <xacro:property name="front_length" value="0.058" />
   <xacro:property name="rear_length" value="0.040" />
@@ -281,4 +282,78 @@
   </link>
   <xacro:enable_self_collision link_name="base_link"/>
+  <link name="imu_link">
+    <visual>
+      <geometry>
+        <box size="${imu_size} ${imu_size} ${imu_size}"/>
+      </geometry>
+      <origin rpy="0 0 0" xyz="0 0 0"/>
+      <material name="grey"/>
+    </visual>
+    <collision>
+      <geometry>
+        <box size="${imu_size} ${imu_size} ${imu_size}"/>
+      </geometry>
+      <origin rpy="0 0 0" xyz="0 0 0"/>
+    </collision>
+    <xacro:box_inertial mass="0.001" x="${imu_size}" y="${imu_size}" z="${imu_size}">
+      <origin rpy="0 0 0" xyz="0 0 0"/>
+    </xacro:box_inertial>
+  </link>
+  <joint name="imu_joint" type="fixed">
+    <parent link="base_link"/>
+    <child link="imu_link"/>
+    <origin rpy="0 0 0" xyz="0 0 0"/>
+  </joint>
+  <gazebo reference="imu_link">
+    <sensor name="imu_sensor" type="imu">
+      <always_on>true</always_on>
+      <update_rate>100</update_rate>
+      <visualize>false</visualize>
+      <topic>imu/data</topic>
+      <gz_frame_id>imu_link</gz_frame_id>
+      <imu>
+        <angular_velocity>
+          <x>
+            <noise type="gaussian">
+              <mean>0.0</mean>
+              <stddev>0.0002</stddev>
+            </noise>
+          </x>
+          <y>
+            <noise type="gaussian">
+              <mean>0.0</mean>
+              <stddev>0.0002</stddev>
+            </noise>
+          </y>
+          <z>
+            <noise type="gaussian">
+              <mean>0.0</mean>
+              <stddev>0.0002</stddev>
+            </noise>
+          </z>
+        </angular_velocity>
+        <linear_acceleration>
+          <x>
+            <noise type="gaussian">
+              <mean>0.0</mean>
+              <stddev>0.017</stddev>
+            </noise>
+          </x>
+          <y>
+            <noise type="gaussian">
+              <mean>0.0</mean>
+              <stddev>0.017</stddev>
+            </noise>
+          </y>
+          <z>
+            <noise type="gaussian">
+              <mean>0.0</mean>
+              <stddev>0.017</stddev>
+            </noise>
+          </z>
+        </linear_acceleration>
+      </imu>
+    </sensor>
+  </gazebo>
   <xacro:if value="$(arg pinned_base)">
     <link name="pinned_world"/>
